File: hardware/v2.0/gpdi.kicad_sch (KiCad schematic)
At the start: 20 parts, among them J2 GPDI_C_1.3, U1 ECP5-CABGA256, U5 TPD2EUSB30A, U6 PCA9306DC1

Commit message: Authoring
Other:
- company: Chengyin Yao (cheyao) -> Chengyin Yao (cheyao), Vadym Vikulin
Changed lines of the file:
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@@
 	(title_block
 		(title "Icepi Zero")
-		(date "2025-10-10")
-		(rev "v1.3")
-		(company "Chengyin Yao (cheyao)")
+		(date "2026-01-05")
+		(rev "v2.0")
+		(company "Chengyin Yao (cheyao), Vadym Vikulin")
 		(comment 1 "https://github.com/cheyao/icepi-zero")
 		(comment 2 "License: Solderpad")
