File: hardware/v1.4-wip/gpdi.kicad_sch (KiCad schematic)
At the start: 20 parts, among them J2 GPDI_C_1.3, U1 ECP5-CABGA256, U5 TPD2EUSB30A, U6 PCA9306DC1

Commit message: Prepare for v1.4 production batch
Parts:
- U5: footprint Package_TO_SOT_SMD:Texas_DRT-3 -> icepi-lib:Texas_DRT-3
Changed lines of the file:
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@@
 		(title "Icepi Zero")
 		(date "2025-10-10")
-		(rev "v1.3")
+		(rev "v1.4")
 		(company "Chengyin Yao (cheyao)")
 		(comment 1 "https://github.com/cheyao/icepi-zero")
@@
 			)
 		)
-		(property "Footprint" "Package_TO_SOT_SMD:Texas_DRT-3"
+		(property "Footprint" "icepi-lib:Texas_DRT-3"
 			(at 167.64 144.78 0)
 			(hide yes)
