File: hardware/v1.4-wip/icepi-zero.kicad_pcb (KiCad board)
At the start: 4 copper layers, 65 x 30 mm, 163 parts, among them J1 Conn_02x20_Counter_Clockwise, J2 GPDI_C_1.3, J3 USB_C_Receptacle_USB2.0_14P, J4 USB_C_Receptacle_USB2.0_14P, J5 USB_C_Receptacle_USB2.0_14P, J6 Micro_SD_Card_Det2, SW1 SW_Push, SW2 SW_Push, U1 ECP5-CABGA256, U10 TPD2EUSB30A, U11 W9825G6KH, U12 W25Q128JVS, U2 TLV62569DBV, U3 TLV62569DBV, U4 TLV62569DBV, U5 TPD2EUSB30A, U6 PCA9306DC1, U7 TPD2EUSB30A, U8 TPD2EUSB30A, U9 FT231XQ, Y1 SG-8018CG 50.000000MHz

Commit message: Prepare for v1.4 production batch
Parts:
- added LOGO1: ~, PCM_ckl-misc:Icy Electronics Logo, B.Cu at (169.2, 102.8)
- C46, C47, C48, C49, C50: value 22nF -> 100nF; footprint Capacitor_SMD:C_0603_1608Metric -> Capacitor_SMD:C_0402_1005Metric
- C51, C52: value 22nF -> 10uF
- R1, R2, R20, R21, R3, R32, R33, R4, R42, R5: value 1k -> 1.1k
- U10, U5, U7, U8: footprint Package_TO_SOT_SMD:Texas_DRT-3 -> icepi-lib:Texas_DRT-3
- moved C48 3.82 mm to (168.3, 109.0), turned to 180 degrees
- moved C50 3.19 mm to (165.8, 112.0), turned to 0 degrees
- moved C47 0.95 mm to (161.9, 111.5)
- moved C49 0.70 mm to (157.5, 110.9)
- moved C46 0.33 mm to (168.9, 97.5)
- moved C8 0.08 mm to (149.1, 106.9)
- moved C31 0.07 mm to (147.2, 106.7)
Routing:
- net +3V3: track 97.2 -> 94.0 mm
- net GND: track 103.4 -> 101.4 mm
- net +1V1: track 40.6 -> 42.1 mm
- net /GPDI/GPDI_HPD: track 27.3 -> 27.9 mm
