File: hardware/v1.4-wip/icepi-zero.kicad_sch (KiCad schematic)
At the start: 29 parts, among them J1 Conn_02x20_Counter_Clockwise, SW1 SW_Push, SW2 SW_Push, U1 ECP5-CABGA256, Y1 SG-8018CG 50.000000MHz

Commit message: Prepare for v1.4 production batch
Parts:
- LOGO1: footprint oshw:OSHW-Certification-Mark-Logo_6x3mm_SilkScreen -> PCM_ckl-misc:Icy Electronics Logo
- R1, R2, R3, R4, R5: value 1k -> 1.1k; LCSC Part # C11702 -> C140223
Changed lines of the file:
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@@
 		(title "Icepi Zero")
 		(date "2025-10-10")
-		(rev "v1.3")
+		(rev "v1.4")
 		(company "Chengyin Yao (cheyao)")
 		(comment 1 "https://github.com/cheyao/icepi-zero")
@@
 			)
 		)
-		(property "Value" "1k"
+		(property "Value" "1.1k"
 			(at 33.02 157.48 90)
 			(show_name no)
@@
 			)
 		)
-		(property "LCSC Part #" "C11702"
+		(property "LCSC Part #" "C140223"
 			(at 33.02 161.29 0)
 			(hide yes)
@@
 			)
 		)
-		(property "Value" "1k"
+		(property "Value" "1.1k"
 			(at 33.02 180.34 90)
 			(show_name no)
@@
 			)
 		)
-		(property "LCSC Part #" "C11702"
+		(property "LCSC Part #" "C140223"
 			(at 33.02 184.15 0)
 			(hide yes)
@@
 			)
 		)
-		(property "Value" "1k"
+		(property "Value" "1.1k"
 			(at 33.02 133.35 90)
 			(show_name no)
@@
 			)
 		)
-		(property "LCSC Part #" "C11702"
+		(property "LCSC Part #" "C140223"
 			(at 33.02 137.16 0)
 			(hide yes)
@@
 			)
 		)
-		(property "Value" "1k"
+		(property "Value" "1.1k"
 			(at 33.02 146.05 90)
 			(show_name no)
@@
 			)
 		)
-		(property "LCSC Part #" "C11702"
+		(property "LCSC Part #" "C140223"
 			(at 33.02 149.86 0)
 			(hide yes)
@@
 			)
 		)
-		(property "Value" "1k"
+		(property "Value" "1.1k"
 			(at 33.02 168.91 90)
 			(show_name no)
@@
 			)
 		)
-		(property "LCSC Part #" "C11702"
+		(property "LCSC Part #" "C140223"
 			(at 33.02 172.72 0)
 			(hide yes)
@@
 		(in_bom no)
 		(on_board yes)
-		(in_pos_files yes)
+		(in_pos_files no)
 		(dnp no)
 		(fields_autoplaced yes)
@@
 			)
 		)
-		(property "Footprint" "oshw:OSHW-Certification-Mark-Logo_6x3mm_SilkScreen"
+		(property "Footprint" "PCM_ckl-misc:Icy Electronics Logo"
 			(at 24.13 20.32 0)
 			(hide yes)
