File: hardware/v1.4-wip/sdram.kicad_sch (KiCad schematic)
At the start: 10 parts, among them U1 ECP5-CABGA256, U11 W9825G6KH

Commit message: Prepare for v1.4 production batch
Parts:
- C46, C47, C48, C49, C50: value 22nF -> 100nF; footprint Capacitor_SMD:C_0603_1608Metric -> Capacitor_SMD:C_0402_1005Metric; LCSC Part # C77571 -> C307331; Manufactuer Part Number 0603B223K500NT -> CL05B104KB54PNC
- C51, C52: value 22nF -> 10uF; LCSC Part # C77571 -> C19702; Manufactuer Part Number 0603B223K500NT -> CL10A106KP8NNNC
