File: hardware/v1.4-wip/usb.kicad_sch (KiCad schematic)
At the start: 48 parts, among them J3 USB_C_Receptacle_USB2.0_14P, J4 USB_C_Receptacle_USB2.0_14P, J5 USB_C_Receptacle_USB2.0_14P, U1 ECP5-CABGA256, U10 TPD2EUSB30A, U7 TPD2EUSB30A, U8 TPD2EUSB30A, U9 FT231XQ

Commit message: Prepare for v1.4 production batch
Parts:
- R20, R21, R32, R33, R42: value 1k -> 1.1k; LCSC Part # C11702 -> C140223
- U10, U7, U8: footprint Package_TO_SOT_SMD:Texas_DRT-3 -> icepi-lib:Texas_DRT-3
Changed lines of the file:
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@@
 		(title "Icepi Zero")
 		(date "2025-10-10")
-		(rev "v1.3")
+		(rev "v1.4")
 		(company "Chengyin Yao (cheyao)")
 		(comment 1 "https://github.com/cheyao/icepi-zero")
@@
 			)
 		)
-		(property "Footprint" "Package_TO_SOT_SMD:Texas_DRT-3"
+		(property "Footprint" "icepi-lib:Texas_DRT-3"
 			(at 48.26 149.86 0)
 			(hide yes)
@@
 			)
 		)
-		(property "Value" "1k"
+		(property "Value" "1.1k"
 			(at 223.52 24.13 90)
 			(show_name no)
@@
 			)
 		)
-		(property "LCSC Part #" "C11702"
+		(property "LCSC Part #" "C140223"
 			(at 223.52 24.13 0)
 			(hide yes)
@@
 			)
 		)
-		(property "Value" "1k"
+		(property "Value" "1.1k"
 			(at 101.6 24.13 90)
 			(show_name no)
@@
 			)
 		)
-		(property "LCSC Part #" "C11702"
+		(property "LCSC Part #" "C140223"
 			(at 101.6 24.13 0)
 			(hide yes)
@@
 			)
 		)
-		(property "Value" "1k"
+		(property "Value" "1.1k"
 			(at 105.41 166.37 90)
 			(show_name no)
@@
 			)
 		)
-		(property "LCSC Part #" "C11702"
+		(property "LCSC Part #" "C140223"
 			(at 105.41 170.18 0)
 			(hide yes)
@@
 			)
 		)
-		(property "Footprint" "Package_TO_SOT_SMD:Texas_DRT-3"
+		(property "Footprint" "icepi-lib:Texas_DRT-3"
 			(at 96.52 72.39 0)
 			(hide yes)
@@
 			)
 		)
-		(property "Footprint" "Package_TO_SOT_SMD:Texas_DRT-3"
+		(property "Footprint" "icepi-lib:Texas_DRT-3"
 			(at 231.14 73.66 0)
 			(hide yes)
@@
 			)
 		)
-		(property "Value" "1k"
+		(property "Value" "1.1k"
 			(at 101.6 77.47 90)
 			(show_name no)
@@
 			)
 		)
-		(property "LCSC Part #" "C11702"
+		(property "LCSC Part #" "C140223"
 			(at 101.6 77.47 0)
 			(hide yes)
@@
 			)
 		)
-		(property "Value" "1k"
+		(property "Value" "1.1k"
 			(at 223.52 77.47 90)
 			(show_name no)
@@
 			)
 		)
-		(property "LCSC Part #" "C11702"
+		(property "LCSC Part #" "C140223"
 			(at 223.52 77.47 0)
 			(hide yes)
