File: hardware/v1.4/flash.kicad_sch (KiCad schematic)
At the start: 11 parts, among them U1 ECP5-CABGA256, U12 W25Q128JVS

Commit message: Consolidated v1.4 version
Parts:
- R48: value 15k -> 4.7k; LCSC Link https://lcsc.com/product-detail/Chip-Resistor-Surface-Mount_UNI-ROYAL-0402WGF1502TCE_C25756.html -> https://lcsc.com/product-detail/Chip-Resistor-Surface-Mount_UNI-ROYAL-0402WGF4701TCE_C25900.html; Manufactuer Part Number 0402WGF1502TCE -> 0402WGF4701TCE
Changed lines of the file:
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@@
 			)
 		)
-		(property "Value" "15k"
+		(property "Value" "4.7k"
 			(at 66.04 64.77 90)
 			(show_name no)
@@
 			)
 		)
-		(property "LCSC Link" "https://lcsc.com/product-detail/Chip-Resistor-Surface-Mount_UNI-ROYAL-0402WGF1502TCE_C25756.html"
+		(property "LCSC Link" "https://lcsc.com/product-detail/Chip-Resistor-Surface-Mount_UNI-ROYAL-0402WGF4701TCE_C25900.html"
 			(at 66.04 64.77 90)
 			(hide yes)
@@
 			)
 		)
-		(property "Manufactuer Part Number" "0402WGF1502TCE"
+		(property "Manufactuer Part Number" "0402WGF4701TCE"
 			(at 66.04 64.77 90)
 			(hide yes)
