File: hardware/v1.4/icepi-zero.kicad_sch (KiCad schematic)
At the start: 29 parts, among them J1 Conn_02x20_Counter_Clockwise, SW1 SW_Push, SW2 SW_Push, U1 ECP5-CABGA256, Y1 SG-8018CG 50.000000MHz

Commit message: Consolidated v1.4 version
Other:
- note added: "Icepi Zero v1.4"
- note removed: "Icepi Zero v1.3!"
Changed lines of the file:
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@@
 		(comment 9 "OSHWA FR000026")
 	)
-	(text "Icepi Zero v1.3!"
+	(text "Icepi Zero v1.4"
 		(exclude_from_sim no)
 		(at 135.89 18.542 0)
